File: neopixels.kicad_sch (KiCad schematic)
At the start: 10 parts

Commit message: Swap FT231XQ for FT231XS
Signed-off-by: Giuseppe Barillari <joe2k01dev@gmail.com>
Connections:
- no-connect marks 0 -> 2
Changed lines of the file:
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@@
   (junction (at 74.93 58.42) (diameter 0) (color 0 0 0 0)
   )
+  (no_connect (at 250.19 50.8))
+  (no_connect (at 250.19 53.34))
   (wire (pts (xy 116.84 58.42) (xy 137.16 58.42))
     (stroke (width 0) (type default) (color 0 0 0 0))
