File: XmasTree.kicad_sch (KiCad schematic)
At the start: 18 parts, among them J1 USB_B_Micro, Q1 BSN20, SW1 SW_Push, U1 FT231XS, U2 AP2202K-3.3

Commit message: Update
Parts:
- gave numbers to parts that had none: 2
Changed lines of the file:
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@@
   (symbol (lib_id "Device:C") (at 106.68 82.55 0) (unit 1)
     (in_bom yes) (on_board yes) (fields_autoplaced)
-    (property "Reference" "C?" (id 0) (at 110.49 81.2799 0)
+    (property "Reference" "C9" (id 0) (at 110.49 81.2799 0)
       (effects (font (size 1.27 1.27)) (justify left))
     )
@@
   (symbol (lib_id "power:GND") (at 106.68 86.36 0) (unit 1)
     (in_bom yes) (on_board yes) (fields_autoplaced)
-    (property "Reference" "#PWR?" (id 0) (at 106.68 92.71 0)
+    (property "Reference" "#PWR0103" (id 0) (at 106.68 92.71 0)
       (effects (font (size 1.27 1.27)) hide)
     )
@@
   (symbol (lib_id "power:GND") (at 62.23 97.79 0) (unit 1)
     (in_bom yes) (on_board yes) (fields_autoplaced)
-    (property "Reference" "#PWR?" (id 0) (at 62.23 104.14 0)
+    (property "Reference" "#PWR0102" (id 0) (at 62.23 104.14 0)
       (effects (font (size 1.27 1.27)) hide)
     )
@@
   (symbol (lib_id "Device:C") (at 62.23 92.71 0) (unit 1)
     (in_bom yes) (on_board yes) (fields_autoplaced)
-    (property "Reference" "C?" (id 0) (at 66.04 91.4399 0)
+    (property "Reference" "C8" (id 0) (at 66.04 91.4399 0)
       (effects (font (size 1.27 1.27)) (justify left))
     )
@@
       (reference "#PWR0101") (unit 1) (value "+3.3V") (footprint "")
     )
+    (path "/8c375b8b-2481-44c3-b896-1da9ebcb5e72"
+      (reference "#PWR0102") (unit 1) (value "GND") (footprint "")
+    )
     (path "/74bcc9d8-e9ac-4aae-9957-6d86ffae2207"
-      (reference "#PWR?") (unit 1) (value "GND") (footprint "")
-    )
-    (path "/8c375b8b-2481-44c3-b896-1da9ebcb5e72"
-      (reference "#PWR?") (unit 1) (value "GND") (footprint "")
+      (reference "#PWR0103") (unit 1) (value "GND") (footprint "")
     )
     (path "/ca8ec33b-f640-4dee-bfae-05e92864f688"
@@
       (reference "C7") (unit 1) (value "10n") (footprint "Capacitor_SMD:C_0805_2012Metric_Pad1.18x1.45mm_HandSolder")
     )
+    (path "/c204358c-67f2-4de0-8610-7251e391bcca"
+      (reference "C8") (unit 1) (value "10n") (footprint "Capacitor_SMD:C_0805_2012Metric_Pad1.18x1.45mm_HandSolder")
+    )
     (path "/0bf5f4dd-88c5-4f7b-b1b3-354b095af0b2"
-      (reference "C?") (unit 1) (value "1u") (footprint "Capacitor_SMD:C_0805_2012Metric_Pad1.18x1.45mm_HandSolder")
-    )
-    (path "/c204358c-67f2-4de0-8610-7251e391bcca"
-      (reference "C?") (unit 1) (value "10n") (footprint "Capacitor_SMD:C_0805_2012Metric_Pad1.18x1.45mm_HandSolder")
+      (reference "C9") (unit 1) (value "1u") (footprint "Capacitor_SMD:C_0805_2012Metric_Pad1.18x1.45mm_HandSolder")
     )
     (path "/c11ac4d5-9454-4a04-af9a-9159635e486a/5a7f9c5d-c505-4a22-94e2-c776ce80000e"
